File: nadeshiko.kicad_pcb (KiCad board)
At the start: 0 parts

Commit message: rev2c
Parts:
- added C1: 3.3nF, Capacitor_SMD:C_0805_2012Metric_Pad1.18x1.45mm_HandSolder, F.Cu at (142.0, 101.5)
- added C2: 3.3nF, Capacitor_SMD:C_0805_2012Metric_Pad1.18x1.45mm_HandSolder, F.Cu at (134.5, 101.5)
- added C3: 3.3nF, Capacitor_SMD:C_0805_2012Metric_Pad1.18x1.45mm_HandSolder, F.Cu at (130.0, 109.5)
- added C4: 47nF, Capacitor_SMD:C_0805_2012Metric_Pad1.18x1.45mm_HandSolder, F.Cu at (156.0, 95.5)
- added D1: 1N4742, Diode_THT:D_DO-41_SOD81_P10.16mm_Horizontal, F.Cu at (122.0, 99.6)
- added D2: 1N4742, Diode_THT:D_DO-41_SOD81_P10.16mm_Horizontal, F.Cu at (127.0, 89.4)
- added J1: 12V_Pin, Connector_PinHeader_2.54mm:PinHeader_1x02_P2.54mm_Vertical, F.Cu at (163.0, 93.2)
- added J2: GND_Pin, Connector_PinHeader_2.54mm:PinHeader_1x02_P2.54mm_Vertical, F.Cu at (163.0, 107.7)
- added J3: OUT_Pin, Connector_PinHeader_2.54mm:PinHeader_1x01_P2.54mm_Vertical, F.Cu at (163.0, 102.5)
- added R1: 10k, Resistor_SMD:R_0805_2012Metric_Pad1.20x1.40mm_HandSolder, F.Cu at (127.5, 84.5)
- added R2: 300k, Resistor_SMD:R_0805_2012Metric_Pad1.20x1.40mm_HandSolder, F.Cu at (132.5, 85.5)
- added R3: 10k, Resistor_SMD:R_0805_2012Metric_Pad1.20x1.40mm_HandSolder, F.Cu at (138.5, 85.5)
- added R4: 10k, Resistor_SMD:R_0805_2012Metric_Pad1.20x1.40mm_HandSolder, F.Cu at (145.0, 84.5)
- added R5: 10k, Resistor_SMD:R_0805_2012Metric_Pad1.20x1.40mm_HandSolder, F.Cu at (150.5, 84.5)
- added R6: 8k, Resistor_SMD:R_0805_2012Metric_Pad1.20x1.40mm_HandSolder, F.Cu at (156.0, 101.5)
- added R7: 1k, Resistor_SMD:R_0805_2012Metric_Pad1.20x1.40mm_HandSolder, F.Cu at (144.0, 109.5)
- added RV1: R_Potentiometer, Potentiometer_THT:Potentiometer_Bourns_3296W_Vertical, F.Cu at (157.0, 109.0)
- added RV2: potentiometer_RK097_Tri, custom_library:potentiometer_RK097_Tri, F.Cu at (137.0, 83.5)
- added SW1: SW_SP3T, Button_Switch_SMD:SW_SP3T_PCM13, F.Cu at (158.7, 88.4)
- added U1: OPA2189, Package_SO:SOIC-8_3.9x4.9mm_P1.27mm, F.Cu at (135.0, 94.0)
- added U2: OPA2189, Package_SO:SOIC-8_3.9x4.9mm_P1.27mm, F.Cu at (148.5, 95.5)
- added U3: TLV1812, Package_TO_SOT_SMD:SOT-23-5_HandSoldering, F.Cu at (137.0, 109.5)
Routing:
- net Net-(U3A-+): track 0.00 -> 93.6 mm, vias 0 -> 3
- net +12V: track 0.00 -> 60.9 mm, vias 0 -> 5
- net Net-(U2A-+): track 0.00 -> 46.1 mm
- net Net-(R7-Pad2): track 0.00 -> 45.3 mm
- net GND: track 0.00 -> 44.2 mm, vias 0 -> 2
- net Net-(U1B-+): track 0.00 -> 38.5 mm, vias 0 -> 2
- net -12V: track 0.00 -> 34.9 mm, vias 0 -> 2
- net Net-(D1-K): track 0.00 -> 30.6 mm, vias 0 -> 2
- net Net-(D1-A): track 0.00 -> 24.6 mm
- net /OUT: track 0.00 -> 24.4 mm, vias 0 -> 1
- net Net-(R3-Pad2): track 0.00 -> 18.8 mm
- net Net-(U1B--): track 0.00 -> 18.1 mm
- net Net-(R4-Pad2): track 0.00 -> 15.6 mm
- net Net-(U2A--): track 0.00 -> 15.4 mm
- net Net-(R5-Pad2): track 0.00 -> 14.1 mm
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- added copper zone on B.Cu, net GND
Other:
- board outline added: 50 x 50 mm
- copper layers 0 -> 2
- board text added: "Project {dblquote}nadeshiko{dblquote} rev2c 111624 ;)"

Commit message: finalize rev2c
Routing:
- net GND: track 44.2 -> 37.4 mm, vias 2 -> 3
- net Net-(U3A-+): track 93.6 -> 99.6 mm
- net +12V: track 60.9 -> 62.6 mm
- net Net-(U1B--): track 18.1 -> 19.1 mm
- net Net-(R3-Pad2): track 18.8 -> 18.2 mm
Other:
- board text added: "Project {dblquote}nadeshiko{dblquote} rev2c ///"
- board text added: "last upd. 241117 Special thanks to Timicasto-chan!!!"
- board text removed: "Project {dblquote}nadeshiko{dblquote} rev2c 111624 ;)"
