File: nadeshiko.kicad_sch (KiCad schematic)
At the start: 19 parts, among them SW1 SW_SP3T, U1 OPA2189, U2 OPA2189, U3 TLV1812

Commit message: rev2c
Parts:
- added J1: 12V_Pin, Connector_PinHeader_2.54mm:PinHeader_1x02_P2.54mm_Vertical, symbol Connector:Conn_01x02_Pin
- added J2: GND_Pin, Connector_PinHeader_2.54mm:PinHeader_1x02_P2.54mm_Vertical, symbol Connector:Conn_01x02_Pin
- added J3: OUT_Pin, Connector_PinHeader_2.54mm:PinHeader_1x01_P2.54mm_Vertical, symbol Connector:Conn_01x01_Pin
- SW1: footprint Button_Switch_SMD:SW_DIP_SPSTx02_Slide_9.78x7.26mm_W8.61mm_P2.54mm -> Button_Switch_SMD:SW_SP3T_PCM13
Connections:
- net +12V: now also J1.1 (Pin_1)
- net -12V: now also J1.2 (Pin_2)
- net GND: now also J2.1 (Pin_1), J2.2 (Pin_2)
- net OUT: now also J3.1 (Pin_1)

Commit message: finalize rev2c
Parts:
- U3: value TLV1812 -> TLV1811; Display TLV1812 -> TLV1811
Changed lines of the file:
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@@
 			)
 		)
-		(property "Value" "TLV1812"
+		(property "Value" "TLV1811"
 			(at 62.23 125.73 0)
 			(effects
@@
 			)
 		)
-		(property "Display" "TLV1812"
+		(property "Display" "TLV1811"
 			(at 64.77 130.8101 0)
 			(effects
@@
 			)
 		)
-		(property "Value" "TLV1812"
+		(property "Value" "TLV1811"
 			(at 63.5 120.65 0)
 			(effects
@@
 			)
 		)
-		(property "Display" "TLV1812"
+		(property "Display" "TLV1811"
 			(at 64.77 106.68 0)
 			(effects
